File: hardware/kicad/motor/Motormodul.kicad_sch (KiCad schematic)
At the start: 42 parts, among them J100 Stapelstecker 2x20, J101 Kettenstecker, Buchse oben, J102 Kettenstecker, Stift unten, J103 Leistungsstecker, Buchse oben, J104 Leistungsstecker, Stift unten, J2 Sensor-Klemme, J3 Notaus-Stiftleiste, J5 Motor-Klemme, Q1 IRF4905, U1 DRV8876PWPR, U100 STM32C011F6P6, U101 SN74LVC1G175, U102 SN74LVC2G00DCUR, U103 SN74LVC1G08, U2 PC817

Commit message: Notaus-Verriegelung wirkte nicht: Diodenklemme durch UND-Gatter ersetzt
Die bisherige Verriegelung (D2 + R14 von NSLEEP auf NOTAUS) hat den
DRV8876-nSLEEP-Pin nie unter seine VIL-Schwelle gezogen. R9 (100 Ohm)
und R14 (1 kOhm) bilden einen Spannungsteiler; der Knoten stand bei
3,05 V, VIL waere 0,8 V (SLVSDS7B, Abschnitt 6.5) -- der Pin lag sogar
ueber VIH. Genau im Auslegungsfall (haengender MCU, GPIO aktiv HIGH)
waere der Motor angeblieben. Der alte Kommentar rechnete nur den
Fehlstrom aus, nicht die Spannung.

Zweiter, unabhaengiger Grund: NOTAUS geht gar nicht auf 0 V, sondern
liegt ueber D3/D4 eine Durchlassspannung ueber Masse. Eine zweite Diode
zum nSLEEP-Pin addiert die naechste -- rund 1,2 V mit 1N4148W, und
selbst mit Schottky auf beiden Wegen bleiben im Grenzfall genau 0,8 V,
also null Reserve. Eine passive Dioden-UND-Verknuepfung kann diese
Schwelle in dieser Topologie nicht sicher einhalten.

Neu: U3 (SN74LVC1G08, LCSC C7832 -- dasselbe Bauteil wie U103, keine
neue Nummer) bildet U1_NSLEEP = NSLEEP AND NOTAUS, dazu C14 als
Abblockkondensator. D2 und R14 entfallen. Gegentaktausgang, damit
0,70 V Reserve gegen VIL bzw. 1,65 V gegen VIH (SCES217AA, 5.5). R9
bleibt bei 100 Ohm und ist jetzt reiner Serienwiderstand vor einem
CMOS-Eingang (II <= 5 uA) -- das Schutzanliegen, fuer das R14 gedacht
war, erledigt sich damit ohne Widerstand.

D3/D4 werden Schottky (BAT54W, SOD-123, LCSC C699107): der gezogene
Ruhepegel des NOTAUS-Busses IST ihre Durchlassspannung, und die eines
1N4148W ist bei diesen Stroemen nicht datenblattbelegt unterhalb 0,8 V.
Mit BAT54W: <= 400 mV (Vishay 86408) bei 2,9 mA im Zehn-Modul-Fall.

tests/test_motormodul.py prueft jetzt PEGEL statt Bauteil-Anwesenheit:
alle Widerstaende und Schwellen liegen als benannte Konstanten mit
Dokument und Abschnitt in motormodul.py, der Test rechnet den Pegel am
nSLEEP-Pin aus dem tatsaechlichen Netzinhalt her und enthaelt fuenf
Gegenproben (alte Klemme, Klemme ohne R14, reine Schottky-Variante,
Si-Koppeld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
Parts:
- removed J100: Stapelstecker 2x20, Connector_PinHeader_2.54mm:PinHeader_2x20_P2.54mm_Vertical, symbol Connector_Generic:Conn_02x20_Odd_Even
- removed J101: Kettenstecker, Buchse oben, Connector_PinHeader_2.54mm:PinHeader_1x02_P2.54mm_Vertical, symbol Connector_Generic:Conn_01x02
- removed Q1: IRF4905, Package_TO_SOT_SMD:TO-252-3_TabPin2, symbol Transistor_FET:IRF4905
- removed R11: 10k, Resistor_SMD:R_0805_2012Metric_Pad1.20x1.40mm_HandSolder, symbol Device:R
- added C14: 0.1u, Capacitor_SMD:C_0805_2012Metric_Pad1.18x1.45mm_HandSolder, symbol Device:C
- added R101: Kennwiderstand (Modultyp), Resistor_SMD:R_0805_2012Metric_Pad1.20x1.40mm_HandSolder, symbol Device:R
- added R105: 10000 (ID_OBEN), Resistor_SMD:R_0805_2012Metric_Pad1.20x1.40mm_HandSolder, symbol Device:R
- added R15: 10k, Resistor_SMD:R_0805_2012Metric_Pad1.20x1.40mm_HandSolder, symbol Device:R
- C10: renamed from R7; value 0.1k -> 0.022u; footprint Resistor_SMD:R_0805_2012Metric_Pad1.20x1.40mm_HandSolder -> Capacitor_SMD:C_0805_2012Metric_Pad1.18x1.45mm_HandSolder; symbol Device:R -> Device:C
- C100: renamed from R102; value 100k -> 100n; footprint Resistor_SMD:R_0805_2012Metric_Pad1.20x1.40mm_HandSolder -> Capacitor_SMD:C_0805_2012Metric_Pad1.18x1.45mm_HandSolder; symbol Device:R -> Device:C
- C101: renamed from U102; value SN74LVC2G00DCUR -> 1000n; footprint Package_SO:VSSOP-8_2.3x2mm_P0.5mm -> Capacitor_SMD:C_0805_2012Metric_Pad1.18x1.45mm_HandSolder; symbol 74xGxx:74LVC2G00 -> Device:C
- C11: renamed from R8; value 0.1k -> 0.1u; footprint Resistor_SMD:R_0805_2012Metric_Pad1.20x1.40mm_HandSolder -> Capacitor_SMD:C_0805_2012Metric_Pad1.18x1.45mm_HandSolder; symbol Device:R -> Device:C
- C12: renamed from C9; value 0.1u -> 220u; footprint Capacitor_SMD:C_0805_2012Metric_Pad1.18x1.45mm_HandSolder -> Capacitor_THT:CP_Radial_D8.0mm_P3.50mm; symbol Device:C -> Device:C_Polarized
- C13: renamed from R6; value 2.2k -> 0.1u; footprint Resistor_SMD:R_0805_2012Metric_Pad1.20x1.40mm_HandSolder -> Capacitor_SMD:C_0805_2012Metric_Pad1.18x1.45mm_HandSolder; symbol Device:R -> Device:C
- D1: renamed from U1; value DRV8876PWPR -> SMCJ30A; footprint DRV8876PWPR:IC_DRV8876PWPR -> Diode_SMD:D_SMC_Handsoldering; symbol DRV8876PWPR:DRV8876PWPR -> Device:D_Zener
- D3: renamed from R14; value 1k -> BAT54W; footprint Resistor_SMD:R_0805_2012Metric_Pad1.20x1.40mm_HandSolder -> Diode_SMD:D_SOD-123; symbol Device:R -> Device:D
- D4: renamed from D2; value 1N4148W -> BAT54W
- J100: renamed from J102; value Kettenstecker, Stift unten -> Stapelstecker 2x20; footprint Connector_PinHeader_2.54mm:PinHeader_1x02_P2.54mm_Vertical -> Connector_PinHeader_2.54mm:PinHeader_2x20_P2.54mm_Vertical; symbol Connector_Generic:Conn_01x02 -> Connector_Generic:Conn_02x20_Odd_Even
- J101: renamed from J103; value Leistungsstecker, Buchse oben -> Kettenstecker, Buchse oben; footprint Connector_PinHeader_2.54mm:PinHeader_2x02_P2.54mm_Vertical -> Connector_PinHeader_2.54mm:PinHeader_1x02_P2.54mm_Vertical; symbol Connector_Generic:Conn_02x02_Odd_Even -> Connector_Generic:Conn_01x02
- J102: renamed from J104; value Leistungsstecker, Stift unten -> Kettenstecker, Stift unten; footprint Connector_PinHeader_2.54mm:PinHeader_2x02_P2.54mm_Vertical -> Connector_PinHeader_2.54mm:PinHeader_1x02_P2.54mm_Vertical; symbol Connector_Generic:Conn_02x02_Odd_Even -> Connector_Generic:Conn_01x02
- J103: renamed from U100; value STM32C011F6P6 -> Leistungsstecker, Buchse oben; footprint Package_SO:TSSOP-20_4.4x6.5mm_P0.65mm -> Connector_PinHeader_2.54mm:PinHeader_2x02_P2.54mm_Vertical; symbol MCU_ST_STM32C0:STM32C011F6Px -> Connector_Generic:Conn_02x02_Odd_Even
- J104: renamed from C100; value 100n -> Leistungsstecker, Stift unten; footprint Capacitor_SMD:C_0805_2012Metric_Pad1.18x1.45mm_HandSolder -> Connector_PinHeader_2.54mm:PinHeader_2x02_P2.54mm_Vertical; symbol Device:C -> Connector_Generic:Conn_02x02_Odd_Even
- J2: renamed from U2; value PC817 -> Sensor-Klemme; footprint Package_SO:SOP-4_3.8x4.1mm_P2.54mm -> TerminalBlock_Phoenix:TerminalBlock_Phoenix_MKDS-3-3-5.08_1x03_P5.08mm_Horizontal; symbol Isolator:PC817 -> Connector:Screw_Terminal_01x03
- J3: renamed from D4; value 1N4148W -> Notaus-Stiftleiste; footprint Diode_SMD:D_SOD-123 -> Connector_PinHeader_2.54mm:PinHeader_1x04_P2.54mm_Vertical; symbol Device:D -> Connector:Conn_01x04_Pin
- J5: renamed from D3; value 1N4148W -> Motor-Klemme; footprint Diode_SMD:D_SOD-123 -> TerminalBlock_Phoenix:TerminalBlock_Phoenix_MKDS-3-2-5.08_1x02_P5.08mm_Horizontal; symbol Device:D -> Connector:Screw_Terminal_01x02
- Q1: renamed from R12; value 10k -> IRF4905; footprint Resistor_SMD:R_0805_2012Metric_Pad1.20x1.40mm_HandSolder -> Package_TO_SOT_SMD:TO-252-3_TabPin2; symbol Device:R -> Transistor_FET:IRF4905
- R10: renamed from J2; value Sensor-Klemme -> 4.7k; footprint TerminalBlock_Phoenix:TerminalBlock_Phoenix_MKDS-3-3-5.08_1x03_P5.08mm_Horizontal -> Resistor_SMD:R_0805_2012Metric_Pad1.20x1.40mm_HandSolder; symbol Connector:Screw_Terminal_01x03 -> Device:R; now not fitted
- R102: renamed from U102; value SN74LVC2G00DCUR -> 100k; footprint Package_SO:VSSOP-8_2.3x2mm_P0.5mm -> Resistor_SMD:R_0805_2012Metric_Pad1.20x1.40mm_HandSolder; symbol 74xGxx:74LVC2G00 -> Device:R
- R11: renamed from D1; value SMCJ30A -> 10k; footprint Diode_SMD:D_SMC_Handsoldering -> Resistor_SMD:R_0805_2012Metric_Pad1.20x1.40mm_HandSolder; symbol Device:D_Zener -> Device:R
- R12: renamed from C12; value 220u -> 10k; footprint Capacitor_THT:CP_Radial_D8.0mm_P3.50mm -> Resistor_SMD:R_0805_2012Metric_Pad1.20x1.40mm_HandSolder; symbol Device:C_Polarized -> Device:R
- R13: renamed from R10; value 4.7k -> 10k; now fitted
- R5: renamed from C13; value 0.1u -> 1.3k; footprint Capacitor_SMD:C_0805_2012Metric_Pad1.18x1.45mm_HandSolder -> Resistor_SMD:R_0805_2012Metric_Pad1.20x1.40mm_HandSolder; symbol Device:C -> Device:R
- R6: renamed from J5; value Motor-Klemme -> 2.2k; footprint TerminalBlock_Phoenix:TerminalBlock_Phoenix_MKDS-3-2-5.08_1x02_P5.08mm_Horizontal -> Resistor_SMD:R_0805_2012Metric_Pad1.20x1.40mm_HandSolder; symbol Connector:Screw_Terminal_01x02 -> Device:R
- R8: renamed from R13; value 10k -> 0.1k
- R9: renamed from R5; value 1.3k -> 0.1k
- U1: renamed from C10; value 0.022u -> DRV8876PWPR; footprint Capacitor_SMD:C_0805_2012Metric_Pad1.18x1.45mm_HandSolder -> DRV8876PWPR:IC_DRV8876PWPR; symbol Device:C -> DRV8876PWPR:DRV8876PWPR
- U100: renamed from U101; value SN74LVC1G175 -> STM32C011F6P6; footprint Package_TO_SOT_SMD:SOT-363_SC-70-6 -> Package_SO:TSSOP-20_4.4x6.5mm_P0.65mm; symbol 74xGxx:74LVC1G175 -> MCU_ST_STM32C0:STM32C011F6Px
- U101: renamed from C101; value 1000n -> SN74LVC1G175; footprint Capacitor_SMD:C_0805_2012Metric_Pad1.18x1.45mm_HandSolder -> Package_TO_SOT_SMD:SOT-363_SC-70-6; symbol Device:C -> 74xGxx:74LVC1G175
- U102: renamed from U103; value SN74LVC1G08 -> SN74LVC2G00DCUR; footprint Package_TO_SOT_SMD:SOT-353_SC-70-5 -> Package_SO:VSSOP-8_2.3x2mm_P0.5mm; symbol 74xGxx:74LVC1G08 -> 74xGxx:74LVC2G00
- U102: renamed from R104; value 10000 (ID_OBEN) -> SN74LVC2G00DCUR; footprint Resistor_SMD:R_0805_2012Metric_Pad1.20x1.40mm_HandSolder -> Package_SO:VSSOP-8_2.3x2mm_P0.5mm; symbol Device:R -> 74xGxx:74LVC2G00
- U103: renamed from R100; value Kennwiderstand (Modultyp) -> SN74LVC1G08; footprint Resistor_SMD:R_0805_2012Metric_Pad1.20x1.40mm_HandSolder -> Package_TO_SOT_SMD:SOT-353_SC-70-5; symbol Device:R -> 74xGxx:74LVC1G08
- U2: renamed from J3; value Notaus-Stiftleiste -> PC817; footprint Connector_PinHeader_2.54mm:PinHeader_1x04_P2.54mm_Vertical -> Package_SO:SOP-4_3.8x4.1mm_P2.54mm; symbol Connector:Conn_01x04_Pin -> Isolator:PC817
- U3: renamed from R15; value 10k -> SN74LVC1G08; footprint Resistor_SMD:R_0805_2012Metric_Pad1.20x1.40mm_HandSolder -> Package_TO_SOT_SMD:SOT-353_SC-70-5; symbol Device:R -> 74xGxx:74LVC1G08
- renumbered C11 to C9, R101 to R100, R105 to R104, R9 to R7
Connections:
- net D2_A is gone; now on net NOTAUS: D3.2 (A), D4.2 (A)
- net +24V: now also C11.2, C9.1, D1.1 (K), J2.1 (Pin_1), Q1.2 (D), U1.11 (VM); no longer C9.2, D1.11 (VM), R10.1 (Pin_1), R11.1 (K), R12.1
- net 3V3: now also C100.2, C101.2, C11.1, C12.2, C13.2, D1.2 (A), J100.13 (Pin_13), J100.18 (Pin_18), J100.23 (Pin_23), J100.28 (Pin_28), J100.3 (Pin_3), J100.33 (Pin_33), J100.36 (Pin_36), J100.38 (Pin_38), J100.8 (Pin_8), J103.2 (Pin_2), J104.4 (Pin_4), J3.2 (Pin_2), J3.4 (Pin_4), R10.2, R102.1, R13.1, U1.15 (GND), U1.16 (PMODE), U1.17 (EXP), U1.5 (VREF), U1.7 (IMODE), U1.9 (PGND), U100.4 (VDD), U101.5 (VCC), U102.4 (GND), U102.8 (VCC), U103.3 (GND), U103.5 (VCC), U2.3, U3.3 (GND), U3.5 (VCC), C14.1, C14.2, R101.2, R105.1, R15.1; no longer C9.1, D1.15 (GND), D1.16 (PMODE), D1.17 (EXP), D1.5 (VREF), D1.7 (IMODE), D1.9 (PGND), J100.2 (Pin_2), J101.4 (Pin_4), J102.4 (Pin_4), J103.5 (VSS), J104.1, J2.2, Q1.2, R10.3 (Pin_3), R11.2 (A), R13.2, R8.1, R9.2, U100.2 (GND), U102.1, U102.3 (GND), U102.4 (GND), U102.5 (VCC), U102.8 (VCC), U103.2, U2.4 (Pin_4), U3.1
- net BOOT0: now also U100.19 (PA14), U103.4; no longer J103.19 (PA14), U102.4
- net CPH: now also C10.1, U1.13 (CPH); no longer D1.13 (CPH), U1.1
- net CPL: now also C10.2, U1.14 (CPL); no longer D1.14 (CPL), U1.2
- net FLASH_MODE: now also J100.5 (Pin_5), U102.5, U103.1; no longer C101.5, U102.1
- net FLASH_RX: now also J100.2 (Pin_2), U100.16 (PA9/PA11); no longer J103.16 (PA9/PA11)
- net FLASH_TX: now also J100.1 (Pin_1), U100.17 (PA10/PA12); no longer J103.17 (PA10/PA12)
- net I2C_SCL: now also J100.7 (Pin_7), U100.20 (PB6); no longer J103.20 (PB6)
- net I2C_SDA: now also J100.6 (Pin_6), U100.1 (PB7); no longer J103.1 (PB7)
- net ID0: now also R100.1, R104.2, U100.7 (PA0); no longer J103.7 (PA0), U102.2, U103.1
- net ID1: now also U100.8 (PA1), R101.1, R105.2; no longer J103.8 (PA1), R100.1, R104.2
- net IN1: now also R7.1, U100.9 (PA2); no longer C10.1, J103.9 (PA2)
- net IN2: now also R8.1, U100.10 (PA3); no longer C11.1, J103.10 (PA3)
- net IPROPI: now also C13.1, R10.1, U1.6 (IPROPI), U100.13 (PA6); no longer D1.6 (IPROPI), J103.13 (PA6), R13.1, R9.1
- net NCLR: now also C101.1, R102.2, U101.6 (~{CLR}); no longer C100.2, U100.6 (~{CLR}), U101.1
- net NFAULT: now also R13.2, U1.4 (~{NFAULT}), U100.12 (PA5); no longer D1.4 (~{NFAULT}), J103.12 (PA5), R8.2
- net NOTAUS: now also J100.9 (Pin_9), R15.2; no longer D4.1 (K), J3.2 (A), J5.2 (A)
- net NOTAUS_1: now also D3.1 (K), J3.1 (Pin_1), U100.3 (PC15); no longer J103.3 (PC15), J5.1 (K), U2.1 (Pin_1)
- net NOTAUS_2: now also D4.1 (K), J3.3 (Pin_3), U100.14 (PA7); no longer J103.14 (PA7), J3.1 (K), U2.3 (Pin_3)
- net NQ: now also U102.6, U102.7; no longer C101.6, R102.7
- net NRST: now also U100.6 (PF2), U102.3; no longer C101.3, J103.6 (PF2)
- net NSLEEP: now also R9.1, U100.11 (PA4); no longer J103.11 (PA4), R7.1
- net Out1: now also J5.1 (Pin_1), U1.8 (OUT1); no longer D1.8 (OUT1), R6.1 (Pin_1)
- net Out2: now also J5.2 (Pin_2), U1.10 (OUT2); no longer D1.10 (OUT2), R6.2 (Pin_2)
- net PWR24V: now also J103.1 (Pin_1), J103.3 (Pin_3), J104.1 (Pin_1), J104.3 (Pin_3), Q1.3 (S), R11.2; no longer J101.1 (Pin_1), J101.3 (Pin_3), J102.1 (Pin_1), J102.3 (Pin_3)
- net Q1_GATE: now also R11.1, R12.1
- net SEL_CLK: now also J100.10 (Pin_10), U101.1 (C); no longer U100.1 (C)
- net SEL_IN: now also J101.1 (Pin_1), U101.3 (D); no longer U100.3 (D)
- net SEL_OUT: now also J102.1 (Pin_1), U101.4 (Q), U102.1, U102.2, U103.2; no longer J100.1 (Pin_1), R102.1, R102.2, U100.4 (Q), U102.2
- net SENSOR24V: now also J2.2 (Pin_2), R6.1; no longer C13.1, R10.2 (Pin_2)
- net SENSOR_3V3: now also U100.2 (PC14), U2.4; no longer J103.2 (PC14), J2.4
- net U1_EN_IN1: now also R7.2, U1.1 (EN/IN1); no longer C10.2, D1.1 (EN/IN1)
- net U1_NSLEEP: now also U1.3 (NSLEEP), U3.4; no longer D1.3 (NSLEEP), D3.1, R7.2
- net U1_PH_IN2: now also R8.2, U1.2 (PH/IN2); no longer C11.2, D1.2 (PH/IN2)
- net U2_LED_A: now also R6.2, U2.1; no longer C13.2, J2.1
- net VCP: now also C9.2, U1.12 (VCP); no longer C12.2, D1.12 (VCP)
- new net NSLEEP_GATTER: R9.2, U3.1
Other:
- moved on the sheet: C9, D4, R100, R104, R7, R8, R9

Commit message: Notaus-Eingang war ein Schliesser: Kabelbruch sah aus wie in Ordnung
Der externe Kontakt an J3 lag als Schliesser gegen GND -- Zumachen hiess
Notaus. Ein gebrochenes Kabel, ein abgezogener Stecker oder eine lose
Klemme waren damit von "alles in Ordnung" nicht zu unterscheiden. Jetzt
Ruhestromprinzip: der Kontakt ist ein Oeffner, im Betrieb geschlossen,
und jede Unterbrechung loest aus.

Je Kanal gehen 24 V ueber 3,3 kOhm hinaus und kommen ueber eine zweite
Ader und weitere 3,3 kOhm in einen PC817 zurueck; dessen Emitter treibt
gegen einen 4,7-kOhm-Pulldown den Knoten SCHLEIFE_1/2 (geschlossen =
HIGH). 24 V statt 3,3 V, weil auf einem langen Museumskabel ein
definierter Strom von 3,5 mA robuster ist als ein hochohmiger Pegel --
und weil ein Optokoppler kein Feldpotential an die Logik laesst.

Der Pulldown kann die wired-OR-Sammelleitung NICHT selbst ziehen: gegen
zehn parallele 10-kOhm-Pullups stuende er bei 2,7 V. Ruhestrom verlangt,
dass Abwesenheit von Strom eine aktive Handlung ausloest -- deshalb
sitzt zwischen Knoten und Bus ein Inverter mit Open-Drain-Ausgang
(SN74LVC1G06, C7828). Die Koppeldioden D3/D4 entfallen dabei: eine Diode
in Reihe zum Open-Drain-Ausgang ergaebe 0,4 + 0,4 = 0,8 V, exakt die
VIL-Schwelle, null Reserve. Ohne sie bleibt es bei 0,4 V Reserve --
zahlengleich mit der bisherigen Schottky-Rechnung, weshalb an U3, R9,
R15 und U1_NSLEEP kein Bauteil und keine Zahl geaendert ist.

Strombegrenzung nach aussen: jede Ader hinter mindestens 3,3 kOhm, also
hoechstens 8,0 mA und 0,211 W in jeden denkbaren Kurzschluss -- deshalb
1206 (250 mW, C26032) und nicht 0805.

J3 bleibt vierpolig, hat aber eine voellig andere Bedeutung. Ein
unbenutzter Kanal muss am Stecker gebrueckt werden (Kanal 1 = Pin 1+2,
Kanal 2 = Pin 3+4), und die Verkabelung des Peche-aux-Canards-Exponats
muss beim Umstieg umgeklemmt werden -- beides als Text im Schaltplan und
als Auflage in hardware/bauteile-1b.md, Beleg 11.

Der Test rechnet die Kette nach, statt Bauteile zu zaehlen: er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
Parts:
- removed D3, D4: BAT54W, Diode_SMD:D_SOD-123, symbol Device:D
- added C15, C16: 0.1u, Capacitor_SMD:C_0805_2012Metric_Pad1.18x1.45mm_HandSolder, symbol Device:C
- added R16, R17, R18, R19: 3.3k, Resistor_SMD:R_1206_3216Metric, symbol Device:R
- added R20, R21: 4.7k, Resistor_SMD:R_0805_2012Metric_Pad1.20x1.40mm_HandSolder, symbol Device:R
- added U4, U5: PC817, Package_SO:SOP-4_3.8x4.1mm_P2.54mm, symbol Isolator:PC817
- added U6, U7: SN74LVC1G06, Package_TO_SOT_SMD:SOT-353_SC-70-5, symbol 74xGxx:74LVC1G06
- J101: value Kettenstecker, Buchse oben -> Kettenstecker, Buchse oben (SMD); footprint Connector_PinHeader_2.54mm:PinHeader_1x02_P2.54mm_Vertical -> Connector_PinSocket_2.54mm:PinSocket_1x02_P2.54mm_Vertical_SMD_Pin1Left
- J102: value Kettenstecker, Stift unten -> Kettenstecker, Stift unten (SMD); footprint Connector_PinHeader_2.54mm:PinHeader_1x02_P2.54mm_Vertical -> Connector_PinHeader_2.54mm:PinHeader_1x02_P2.54mm_Vertical_SMD_Pin1Left
- J103: value Leistungsstecker, Buchse oben -> Leistungsstecker, Buchse oben (SMD); footprint Connector_PinHeader_2.54mm:PinHeader_2x02_P2.54mm_Vertical -> Connector_PinSocket_2.54mm:PinSocket_2x02_P2.54mm_Vertical_SMD
- J104: value Leistungsstecker, Stift unten -> Leistungsstecker, Stift unten (SMD); footprint Connector_PinHeader_2.54mm:PinHeader_2x02_P2.54mm_Vertical -> Connector_PinHeader_2.54mm:PinHeader_2x02_P2.54mm_Vertical_SMD
- J3: value Notaus-Stiftleiste -> Notaus-Ruhestrom
Connections:
- net +24V: now also R16.1, R17.1
- net 3V3: now also C15.1, C15.2, C16.1, C16.2, R20.2, R21.2, U4.2, U4.4, U5.2, U5.4, U6.3 (GND), U6.5 (VCC), U7.3 (GND), U7.5 (VCC); no longer J3.2 (Pin_2), J3.4 (Pin_4)
- net NOTAUS: now also U6.4, U7.4
- net NOTAUS_1 renamed KREIS1_A
- net KREIS1_A: now also R16.2; no longer U100.3 (PC15)
- net NOTAUS_2 renamed KREIS2_A
- net KREIS2_A: now also R17.2; no longer U100.14 (PA7)
- new net KREIS1_B: J3.2 (Pin_2), R18.1
- new net KREIS2_B: J3.4 (Pin_4), R19.1
- new net SCHLEIFE_1: R20.1, U100.3 (PC15), U4.3, U6.2
- new net SCHLEIFE_2: R21.1, U100.14 (PA7), U5.3, U7.2
- new net U4_LED_A: R18.2, U4.1
- new net U5_LED_A: R19.2, U5.1
Other:
- note added: "ALTE VERKABELUNG (Schliesser gegen GND) NICHT weiterverwenden: umklemmen."
- note added: "J3 = Notaus, Ruhestrom (OEFFNER): Kanal 1 = Pin 1+2, Kanal 2 = Pin 3+4."
- note added: "UNBENUTZTEN KANAL BRUECKEN (Jumper 2,54 mm) -- sonst meldet er dauerhaft Notaus."

Commit message: Geerbte Fehler aus dem Muttern-Print als Gattung geprueft, drei gefunden
Die Endstufe wurde uebernommen, ohne sie nachzurechnen. Zwei Fehler waren
bekannt, den dritten hat erst die Gattungspruefung gefunden:

R6 (Vorwiderstand des Sensor-Optokopplers) verheizte 0,236 W in einem
0805 mit 0,125 W Belastbarkeit -- Faktor 1,9 dauerhaft ueber Grenzwert.
Behoben nicht durch ein groesseres Gehaeuse, sondern durch Weglassen des
ganzen Sensoreingangs (J2, R6, U2): er war schon im Altprojekt unbenutzt,
und die Spec nennt fuer den Modultyp Motor nur Treiber, Strommessung und
Notaus. Ein Bauteil, das nichts tut, aber ueberlastet ist, wird nicht
vergroessert. Frei wird dabei PC14 als GPIO und der einzige Punkt, an dem
24 V ungeschuetzt Richtung Optokoppler gingen.

Der Optokoppler-Footprint hatte seine Padreihen 5,5 mm auseinander, das
beschaffte Bauteil hat 10,0 mm Anschlussspanne -- die Pads lagen
vollstaendig NEBEN den Anschluessen. Jetzt Pad fuer Pad aus dem
Sharp-Datenblatt gezeichnet, als projekteigene Bibliothek.

DRITTER FALL, von der Gattungspruefung gefunden: Q1 trug "IRF4905" im
TO-252-Footprint. Den IRF4905 gibt es nur als TO-220AB und als D2Pak --
kein TO-252. JLCPCB haette ein anderes Bauteil bestueckt oder gar keins.
Ersetzt durch IRFR5305PbF, derselbe HEXFET-Typ in genau dieser Bauform.

Beide Pruefungen decken jetzt die Klasse: jede Bauform bringt ihre
Belastbarkeit als benannte Groesse mit Herkunft mit (20 Widerstaende
nachgerechnet, 6 davon ueber 5 V), jedes Bauteil braucht einen belegten
Gehaeuseeintrag (35 geometrisch nachgemessen, 14 nach Polzahl und
Bauform). Ein neues Bauteil ohne Beleg faellt durch, nicht erst das
naechste Exemplar desselben Fehlers.

Co-Authored-By: Claude Opus 5 (1M context) <noreply@anthropic.com>
Parts:
- removed C14, C15, C16: 0.1u, Capacitor_SMD:C_0805_2012Metric_Pad1.18x1.45mm_HandSolder, symbol Device:C
- removed J3: Notaus-Ruhestrom, Connector_PinHeader_2.54mm:PinHeader_1x04_P2.54mm_Vertical, symbol Connector:Conn_01x04_Pin
- removed J5: Motor-Klemme, TerminalBlock_Phoenix:TerminalBlock_Phoenix_MKDS-3-2-5.08_1x02_P5.08mm_Horizontal, symbol Connector:Screw_Terminal_01x02
- removed R15: 10k, Resistor_SMD:R_0805_2012Metric_Pad1.20x1.40mm_HandSolder, symbol Device:R
- removed R16, R17, R18, R19: 3.3k, Resistor_SMD:R_1206_3216Metric, symbol Device:R
- removed R20, R21: 4.7k, Resistor_SMD:R_0805_2012Metric_Pad1.20x1.40mm_HandSolder, symbol Device:R
- removed R6: 2.2k, Resistor_SMD:R_0805_2012Metric_Pad1.20x1.40mm_HandSolder, symbol Device:R
- removed U2, U4, U5: PC817, Package_SO:SOP-4_3.8x4.1mm_P2.54mm, symbol Isolator:PC817
- removed U3: SN74LVC1G08, Package_TO_SOT_SMD:SOT-353_SC-70-5, symbol 74xGxx:74LVC1G08
- removed U6, U7: SN74LVC1G06, Package_TO_SOT_SMD:SOT-353_SC-70-5, symbol 74xGxx:74LVC1G06
- added C100: 100n, Capacitor_SMD:C_0805_2012Metric_Pad1.18x1.45mm_HandSolder, symbol Device:C
- added C101: 1000n, Capacitor_SMD:C_0805_2012Metric_Pad1.18x1.45mm_HandSolder, symbol Device:C
- added C13: 0.1u, Capacitor_SMD:C_0805_2012Metric_Pad1.18x1.45mm_HandSolder, symbol Device:C
- added J100: Stapelstecker 2x20, Connector_PinHeader_2.54mm:PinHeader_2x20_P2.54mm_Vertical, symbol Connector_Generic:Conn_02x20_Odd_Even
- added J101: Kettenstecker, Buchse oben (SMD), Connector_PinSocket_2.54mm:PinSocket_1x02_P2.54mm_Vertical_SMD_Pin1Left, symbol Connector_Generic:Conn_01x02
- added J104: Leistungsstecker, Stift unten (SMD), Connector_PinHeader_2.54mm:PinHeader_2x02_P2.54mm_Vertical_SMD, symbol Connector_Generic:Conn_02x02_Odd_Even
- added R10: 4.7k, Resistor_SMD:R_0805_2012Metric_Pad1.20x1.40mm_HandSolder, symbol Device:R
- added R100: Kennwiderstand (Modultyp), Resistor_SMD:R_0805_2012Metric_Pad1.20x1.40mm_HandSolder, symbol Device:R
- added R102: 100k, Resistor_SMD:R_0805_2012Metric_Pad1.20x1.40mm_HandSolder, symbol Device:R
- added R104: 10000 (ID_OBEN), Resistor_SMD:R_0805_2012Metric_Pad1.20x1.40mm_HandSolder, symbol Device:R
- added U100: STM32C011F6P6, Package_SO:TSSOP-20_4.4x6.5mm_P0.65mm, symbol MCU_ST_STM32C0:STM32C011F6Px
- added U101: SN74LVC1G175, Package_TO_SOT_SMD:SOT-363_SC-70-6, symbol 74xGxx:74LVC1G175
- added U102: SN74LVC2G00DCUR, Package_SO:VSSOP-8_2.3x2mm_P0.5mm, symbol 74xGxx:74LVC2G00
- added U103: SN74LVC1G08, Package_TO_SOT_SMD:SOT-353_SC-70-5, symbol 74xGxx:74LVC1G08
- C10: renamed from U102; value SN74LVC2G00DCUR -> 0.022u; footprint Package_SO:VSSOP-8_2.3x2mm_P0.5mm -> Capacitor_SMD:C_0805_2012Metric_Pad1.18x1.45mm_HandSolder; symbol 74xGxx:74LVC2G00 -> Device:C
- C11, C9: renamed from U102; value SN74LVC2G00DCUR -> 0.1u; footprint Package_SO:VSSOP-8_2.3x2mm_P0.5mm -> Capacitor_SMD:C_0805_2012Metric_Pad1.18x1.45mm_HandSolder; symbol 74xGxx:74LVC2G00 -> Device:C
- C12: renamed from R102; value 100k -> 220u; footprint Resistor_SMD:R_0805_2012Metric_Pad1.20x1.40mm_HandSolder -> Capacitor_THT:CP_Radial_D8.0mm_P3.50mm; symbol Device:R -> Device:C_Polarized
- C14: renamed from R12; value 10k -> 0.1u; footprint Resistor_SMD:R_0805_2012Metric_Pad1.20x1.40mm_HandSolder -> Capacitor_SMD:C_0805_2012Metric_Pad1.18x1.45mm_HandSolder; symbol Device:R -> Device:C
- C15: renamed from R8; value 0.1k -> 0.1u; footprint Resistor_SMD:R_0805_2012Metric_Pad1.20x1.40mm_HandSolder -> Capacitor_SMD:C_0805_2012Metric_Pad1.18x1.45mm_HandSolder; symbol Device:R -> Device:C
- C16: renamed from J2; value Sensor-Klemme -> 0.1u; footprint TerminalBlock_Phoenix:TerminalBlock_Phoenix_MKDS-3-3-5.08_1x03_P5.08mm_Horizontal -> Capacitor_SMD:C_0805_2012Metric_Pad1.18x1.45mm_HandSolder; symbol Connector:Screw_Terminal_01x03 -> Device:C
- D1: renamed from U101; value SN74LVC1G175 -> SMCJ30A; footprint Package_TO_SOT_SMD:SOT-363_SC-70-6 -> Diode_SMD:D_SMC_Handsoldering; symbol 74xGxx:74LVC1G175 -> Device:D_Zener
- J3: renamed from C12; value 220u -> Notaus-Ruhestrom; footprint Capacitor_THT:CP_Radial_D8.0mm_P3.50mm -> Connector_PinHeader_2.54mm:PinHeader_1x04_P2.54mm_Vertical; symbol Device:C_Polarized -> Connector:Conn_01x04_Pin
- J5: renamed from Q1; value IRF4905 -> Motor-Klemme; footprint Package_TO_SOT_SMD:TO-252-3_TabPin2 -> TerminalBlock_Phoenix:TerminalBlock_Phoenix_MKDS-3-2-5.08_1x02_P5.08mm_Horizontal; symbol Transistor_FET:IRF4905 -> Connector:Screw_Terminal_01x02
- Q1: renamed from J104; value Leistungsstecker, Stift unten (SMD) -> IRFR5305; footprint Connector_PinHeader_2.54mm:PinHeader_2x02_P2.54mm_Vertical_SMD -> Package_TO_SOT_SMD:TO-252-3_TabPin2; symbol Connector_Generic:Conn_02x02_Odd_Even -> Transistor_FET:Q_PMOS_GDS
- R101: renamed from J101; value Kettenstecker, Buchse oben (SMD) -> Kennwiderstand (Modultyp); footprint Connector_PinSocket_2.54mm:PinSocket_1x02_P2.54mm_Vertical_SMD_Pin1Left -> Resistor_SMD:R_0805_2012Metric_Pad1.20x1.40mm_HandSolder; symbol Connector_Generic:Conn_01x02 -> Device:R
- R105: renamed from J100; value Stapelstecker 2x20 -> 10000 (ID_OBEN); footprint Connector_PinHeader_2.54mm:PinHeader_2x20_P2.54mm_Vertical -> Resistor_SMD:R_0805_2012Metric_Pad1.20x1.40mm_HandSolder; symbol Connector_Generic:Conn_02x20_Odd_Even -> Device:R
- R11: renamed from U100; value STM32C011F6P6 -> 10k; footprint Package_SO:TSSOP-20_4.4x6.5mm_P0.65mm -> Resistor_SMD:R_0805_2012Metric_Pad1.20x1.40mm_HandSolder; symbol MCU_ST_STM32C0:STM32C011F6Px -> Device:R
- R12: renamed from C100; value 100n -> 10k; footprint Capacitor_SMD:C_0805_2012Metric_Pad1.18x1.45mm_HandSolder -> Resistor_SMD:R_0805_2012Metric_Pad1.20x1.40mm_HandSolder; symbol Device:C -> Device:R
- R13: renamed from R105; value 10000 (ID_OBEN) -> 10k
- R15: renamed from D1; value SMCJ30A -> 10k; footprint Diode_SMD:D_SMC_Handsoldering -> Resistor_SMD:R_0805_2012Metric_Pad1.20x1.40mm_HandSolder; symbol Device:D_Zener -> Device:R
- R16: renamed from U1; value DRV8876PWPR -> 3.3k; footprint DRV8876PWPR:IC_DRV8876PWPR -> Resistor_SMD:R_1206_3216Metric; symbol DRV8876PWPR:DRV8876PWPR -> Device:R
- R17: renamed from R9; value 0.1k -> 3.3k; footprint Resistor_SMD:R_0805_2012Metric_Pad1.20x1.40mm_HandSolder -> Resistor_SMD:R_1206_3216Metric
- R18: renamed from C9; value 0.1u -> 3.3k; footprint Capacitor_SMD:C_0805_2012Metric_Pad1.18x1.45mm_HandSolder -> Resistor_SMD:R_1206_3216Metric; symbol Device:C -> Device:R
- R19: renamed from R13; value 10k -> 3.3k; footprint Resistor_SMD:R_0805_2012Metric_Pad1.20x1.40mm_HandSolder -> Resistor_SMD:R_1206_3216Metric
- R20: renamed from C11; value 0.1u -> 4.7k; footprint Capacitor_SMD:C_0805_2012Metric_Pad1.18x1.45mm_HandSolder -> Resistor_SMD:R_0805_2012Metric_Pad1.20x1.40mm_HandSolder; symbol Device:C -> Device:R
- R21: renamed from R10; now fitted
- R5: renamed from R101; value Kennwiderstand (Modultyp) -> 1.3k
- R7: renamed from U103; value SN74LVC1G08 -> 0.1k; footprint Package_TO_SOT_SMD:SOT-353_SC-70-5 -> Resistor_SMD:R_0805_2012Metric_Pad1.20x1.40mm_HandSolder; symbol 74xGxx:74LVC1G08 -> Device:R
- R8: renamed from R104; value 10000 (ID_OBEN) -> 0.1k
- R9: renamed from R100; value Kennwiderstand (Modultyp) -> 0.1k
- U1: renamed from C101; value 1000n -> DRV8876PWPR; footprint Capacitor_SMD:C_0805_2012Metric_Pad1.18x1.45mm_HandSolder -> DRV8876PWPR:IC_DRV8876PWPR; symbol Device:C -> DRV8876PWPR:DRV8876PWPR
- U3: renamed from R11; value 10k -> SN74LVC1G08; footprint Resistor_SMD:R_0805_2012Metric_Pad1.20x1.40mm_HandSolder -> Package_TO_SOT_SMD:SOT-353_SC-70-5; symbol Device:R -> 74xGxx:74LVC1G08
- U4: renamed from C10; value 0.022u -> PC817; footprint Capacitor_SMD:C_0805_2012Metric_Pad1.18x1.45mm_HandSolder -> Optocoupler_PC817:PC817_SMT_Gullwing; symbol Device:C -> Isolator:PC817
- U5: renamed from R5; value 1.3k -> PC817; footprint Resistor_SMD:R_0805_2012Metric_Pad1.20x1.40mm_HandSolder -> Optocoupler_PC817:PC817_SMT_Gullwing; symbol Device:R -> Isolator:PC817
- U6: renamed from R7; value 0.1k -> SN74LVC1G06; footprint Resistor_SMD:R_0805_2012Metric_Pad1.20x1.40mm_HandSolder -> Package_TO_SOT_SMD:SOT-353_SC-70-5; symbol Device:R -> 74xGxx:74LVC1G06
- U7: renamed from C13; value 0.1u -> SN74LVC1G06; footprint Capacitor_SMD:C_0805_2012Metric_Pad1.18x1.45mm_HandSolder -> Package_TO_SOT_SMD:SOT-353_SC-70-5; symbol Device:C -> 74xGxx:74LVC1G06
Connections:
- net SENSOR24V is gone; now on net 3V3: C16.2
- net SENSOR_3V3 is gone; now on net PWR24V: R11.2
- net +24V: now also C11.2, C12.1, C9.1, D1.1 (K), Q1.2 (D), R16.1, R17.1, U1.11 (VM); no longer C16.1 (Pin_1), J3.1, J5.2 (D), R15.1 (K), R16.11 (VM), R18.1, R20.2
- net 3V3: now also C11.1, C12.2, C14.1, C15.1, C15.2, C16.1, R105.1, R15.1, R20.2, U1.15 (GND), U1.16 (PMODE), U1.17 (EXP), U1.5 (VREF), U1.7 (IMODE), U1.9 (PGND), U3.3 (GND), U3.5 (VCC), U4.2, U4.4, U5.4, U6.3 (GND), U6.5 (VCC), U7.3 (GND), U7.5 (VCC), C100.1, C100.2, C101.2, C13.2, J100.13 (Pin_13), J100.18 (Pin_18), J100.23 (Pin_23), J100.28 (Pin_28), J100.3 (Pin_3), J100.33 (Pin_33), J100.36 (Pin_36), J100.38 (Pin_38), J100.8 (Pin_8), J101.2 (Pin_2), J104.2 (Pin_2), J104.4 (Pin_4), R10.2, R100.2, R102.1, R104.1, U100.4 (VDD), U100.5 (VSS), U101.2 (GND), U101.5 (VCC), U102.4 (GND), U102.8 (VCC), U103.3 (GND), U103.5 (VCC); no longer C11.4 (GND), C11.8 (VCC), C12.1, C16.3 (Pin_3), D1.5 (VCC), J3.2, Q1.2 (Pin_2), Q1.4 (Pin_4), R105.13 (Pin_13), R105.18 (Pin_18), R105.23 (Pin_23), R105.28 (Pin_28), R105.3 (Pin_3), R105.33 (Pin_33), R105.36 (Pin_36), R105.38 (Pin_38), R105.8 (Pin_8), R11.4 (VDD), R11.5 (VSS), R12.1, R15.2 (A), R16.15 (GND), R16.16 (PMODE), R16.17 (EXP), R16.5 (VREF), R16.7 (IMODE), R16.9 (PGND), R19.1, R20.1, R7.3 (GND), R7.5 (VCC), R8.1, R9.2, U1.2, U7.2
- net BOOT0: now also U100.19 (PA14), U103.4; no longer R11.19 (PA14), R7.4
- net CPH: now also C10.1, U1.13 (CPH); no longer R16.13 (CPH), U4.1
- net CPL: now also C10.2, U1.14 (CPL); no longer R16.14 (CPL), U4.2
- net FLASH_MODE: now also J100.5 (Pin_5), U102.5, U103.1; no longer C10.5, R105.5 (Pin_5), R7.1
- net FLASH_RX: now also J100.2 (Pin_2), U100.16 (PA9/PA11); no longer R105.2 (Pin_2), R11.16 (PA9/PA11)
- net FLASH_TX: now also J100.1 (Pin_1), U100.17 (PA10/PA12); no longer R105.1 (Pin_1), R11.17 (PA10/PA12)
- net I2C_SCL: now also J100.7 (Pin_7), U100.20 (PB6); no longer R105.7 (Pin_7), R11.20 (PB6)
- net I2C_SDA: now also J100.6 (Pin_6), U100.1 (PB7); no longer R105.6 (Pin_6), R11.1 (PB7)
- net ID0: now also R100.1, R104.2, U100.7 (PA0); no longer R11.7 (PA0), R8.2, R9.1
- net ID1: now also R101.1, R105.2, U100.8 (PA1); no longer R11.8 (PA1), R13.2, R5.1
- net IN1: now also R7.1, U100.9 (PA2); no longer R11.9 (PA2), U6.1
- net IN2: now also R8.1, U100.10 (PA3); no longer C15.1, R11.10 (PA3)
- net IPROPI: now also R5.1, U1.6 (IPROPI), C13.1, R10.1, U100.13 (PA6); no longer R11.13 (PA6), R16.6 (IPROPI), R21.1, U5.1, U7.1
- net KREIS1_A: now also J3.1 (Pin_1), R16.2
- net KREIS1_B: now also J3.2 (Pin_2), R18.1
- net KREIS2_A: now also J3.3 (Pin_3), R17.2
- net KREIS2_B: now also J3.4 (Pin_4), R19.1
- net NCLR: now also C101.1, R102.2, U101.6 (~{CLR}); no longer C12.2, D1.6 (~{CLR}), U1.1
- net NFAULT: now also R13.2, U1.4 (~{NFAULT}), U100.12 (PA5); no longer R11.12 (PA5), R16.4 (~{NFAULT}), R19.2
- net NOTAUS: now also R15.2, U3.2, U6.4, U7.4, J100.9 (Pin_9); no longer R105.9 (Pin_9)
- net NQ: now also U102.6, U102.7; no longer C10.6, C9.7
- net NRST: now also U100.6 (PF2), U102.3; no longer C10.3, R11.6 (PF2)
- net NSLEEP: now also R9.1, U100.11 (PA4); no longer R11.11 (PA4), R17.1
- net NSLEEP_GATTER: now also R9.2, U3.1; no longer R17.2
- net Out1: now also J5.1 (Pin_1), U1.8 (OUT1); no longer R16.8 (OUT1)
- net Out2: now also J5.2 (Pin_2), U1.10 (OUT2); no longer R16.10 (OUT2)
- net PWR24V: now also J104.1 (Pin_1), J104.3 (Pin_3); no longer J5.3 (S), Q1.1 (Pin_1), U3.2
- net Q1_GATE: now also Q1.1 (G), R11.1, R12.1; no longer C14.1, J5.1 (G), U3.1
- net SCHLEIFE_1: now also R20.1, U4.3, U6.2, U100.3 (PC15); no longer R11.3 (PC15)
- net SCHLEIFE_2: now also R21.1, U5.3, U7.2, U100.14 (PA7); no longer R11.14 (PA7)
- net SEL_CLK: now also J100.10 (Pin_10), U101.1 (C); no longer D1.1 (C), R105.10 (Pin_10)
- net SEL_IN: now also J101.1 (Pin_1), U101.3 (D); no longer D1.3 (D), R101.1 (Pin_1)
- net SEL_OUT: now also U101.4 (Q), U102.1, U102.2, U103.2; no longer C9.1, C9.2, D1.4 (Q), R7.2
- net U1_EN_IN1: now also R7.2, U1.1 (EN/IN1); no longer R16.1 (EN/IN1), U6.2
- net U1_NSLEEP: now also U1.3 (NSLEEP), U3.4; no longer R16.3 (NSLEEP)
- net U1_PH_IN2: now also R8.2, U1.2 (PH/IN2); no longer C15.2, R16.2 (PH/IN2)
- net U4_LED_A: now also R18.2, U4.1
- net U5_LED_A: now also R19.2, U5.1
- net VCP: now also C9.2, U1.12 (VCP); no longer R16.12 (VCP), R18.2
- no-connect marks 26 -> 27
Other:
- moved on the sheet: R13, R17, R19, R5, R8, R9
